File: Proyecto/Esquematico.brd (EAGLE design)
At the start: 70.8 x 53.3 mm, 12 parts

Commit message: Se corrigieron algunas pistas
Parts:
- moved R3 2.54 mm to (47.0, 20.3)
- renumbered JP1 to ENCODER, JP2 to 12VIN, JP3 to MOTOR
Routing:
- net N$2: track 63.4 -> 67.8 mm
- net N$11: track 45.5 -> 48.8 mm
- net N$1: track 3.81 -> 6.35 mm
- net N$9: track 24.3 -> 26.5 mm
- net N$4: track 28.2 -> 29.1 mm
- net N$3: track 64.6 -> 65.4 mm
- net N$12: track 28.9 -> 28.3 mm
