File: Proyecto/Esquematico.sch (EAGLE design)
At the start: 12 parts

Commit message: Se corrigieron algunas pistas
Parts:
- renumbered JP1 to ENCODER, JP2 to 12VIN, JP3 to MOTOR
Other:
- note added: "Reemplazar el MOSFET por el modelo correcto"
Changed lines of the file:
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@@
 <part name="U$1" library="adafruit" deviceset="ARDUINO" device="-NOHOLE"/>
 <part name="T1" library="transistor" deviceset="*-NPN-" device="SOT23-BEC" technology="BC817-40LT1"/>
-<part name="JP1" library="adafruit" deviceset="PINHD-1X3" device="CB"/>
+<part name="ENCODER" library="adafruit" deviceset="PINHD-1X3" device="CB"/>
 <part name="T2" library="zetex" deviceset="NMOSSOT223" device=""/>
 <part name="D1" library="diode" deviceset="MBRA340T3" device=""/>
@@
 <part name="R4" library="rcl" deviceset="R-EU_" device="R1206" value="1K"/>
 <part name="R5" library="rcl" deviceset="R-EU_" device="R1206" value="1K"/>
-<part name="JP2" library="pinhead" deviceset="PINHD-1X2" device=""/>
-<part name="JP3" library="pinhead" deviceset="PINHD-1X2" device=""/>
+<part name="12VIN" library="pinhead" deviceset="PINHD-1X2" device=""/>
+<part name="MOTOR" library="pinhead" deviceset="PINHD-1X2" device=""/>
 </parts>
 <sheets>
 <sheet>
 <plain>
+<text x="35.56" y="76.2" size="1.778" layer="91">Reemplazar el MOSFET por el modelo correcto</text>
 </plain>
 <instances>
 <instance part="U$1" gate="G$1" x="35.56" y="22.86"/>
 <instance part="T1" gate="G$1" x="12.7" y="60.96"/>
-<instance part="JP1" gate="A" x="-10.16" y="53.34"/>
+<instance part="ENCODER" gate="A" x="-10.16" y="53.34"/>
 <instance part="T2" gate="A" x="121.92" y="33.02"/>
 <instance part="D1" gate="G$1" x="132.08" y="48.26" rot="R90"/>
@@
 <instance part="R4" gate="G$1" x="15.24" y="76.2" rot="R90"/>
 <instance part="R5" gate="G$1" x="106.68" y="30.48" rot="R180"/>
-<instance part="JP2" gate="G$1" x="114.3" y="63.5"/>
-<instance part="JP3" gate="G$1" x="114.3" y="45.72"/>
+<instance part="12VIN" gate="G$1" x="114.3" y="63.5"/>
+<instance part="MOTOR" gate="G$1" x="114.3" y="45.72"/>
 </instances>
 <busses>
@@
 <pinref part="R3" gate="G$1" pin="2"/>
 <wire x1="-20.32" y1="45.72" x2="-20.32" y2="50.8" width="0.1524" layer="91"/>
-<pinref part="JP1" gate="A" pin="3"/>
+<pinref part="ENCODER" gate="A" pin="3"/>
 <wire x1="-20.32" y1="50.8" x2="-12.7" y2="50.8" width="0.1524" layer="91"/>
 </segment>
@@
 <wire x1="144.78" y1="22.86" x2="121.92" y2="22.86" width="0.1524" layer="91"/>
 <junction x="121.92" y="22.86"/>
-<pinref part="JP2" gate="G$1" pin="2"/>
+<pinref part="12VIN" gate="G$1" pin="2"/>
 <wire x1="111.76" y1="63.5" x2="109.22" y2="63.5" width="0.1524" layer="91"/>
 <wire x1="109.22" y1="63.5" x2="109.22" y2="58.42" width="0.1524" layer="91"/>
@@
 <net name="N$3" class="0">
 <segment>
-<pinref part="JP1" gate="A" pin="2"/>
+<pinref part="ENCODER" gate="A" pin="2"/>
 <wire x1="-12.7" y1="53.34" x2="0" y2="53.34" width="0.1524" layer="91"/>
 <wire x1="0" y1="53.34" x2="0" y2="48.26" width="0.1524" layer="91"/>
@@
 <net name="N$4" class="0">
 <segment>
-<pinref part="JP1" gate="A" pin="1"/>
+<pinref part="ENCODER" gate="A" pin="1"/>
 <wire x1="-12.7" y1="55.88" x2="-12.7" y2="60.96" width="0.1524" layer="91"/>
 <pinref part="R2" gate="G$1" pin="1"/>
@@
 <wire x1="129.54" y1="43.18" x2="132.08" y2="43.18" width="0.1524" layer="91"/>
 <wire x1="132.08" y1="43.18" x2="132.08" y2="45.72" width="0.1524" layer="91"/>
-<pinref part="JP3" gate="G$1" pin="2"/>
+<pinref part="MOTOR" gate="G$1" pin="2"/>
 <wire x1="111.76" y1="45.72" x2="111.76" y2="43.18" width="0.1524" layer="91"/>
 <wire x1="111.76" y1="43.18" x2="119.38" y2="43.18" width="0.1524" layer="91"/>
@@
 <wire x1="124.46" y1="55.88" x2="121.92" y2="55.88" width="0.1524" layer="91"/>
 <wire x1="121.92" y1="55.88" x2="121.92" y2="50.8" width="0.1524" layer="91"/>
-<pinref part="JP3" gate="G$1" pin="1"/>
+<pinref part="MOTOR" gate="G$1" pin="1"/>
 <wire x1="111.76" y1="48.26" x2="111.76" y2="50.8" width="0.1524" layer="91"/>
 <wire x1="111.76" y1="50.8" x2="121.92" y2="50.8" width="0.1524" layer="91"/>
-<pinref part="JP2" gate="G$1" pin="1"/>
+<pinref part="12VIN" gate="G$1" pin="1"/>
 <wire x1="111.76" y1="66.04" x2="111.76" y2="71.12" width="0.1524" layer="91"/>
 <wire x1="111.76" y1="71.12" x2="116.84" y2="71.12" width="0.1524" layer="91"/>
